File: SoilMoistureIoT.kicad_sch (KiCad schematic)
At the start: 0 parts

Commit message: adding some component
Other:
- added sheet mcu (mcu.kicad_sch)
- added sheet modem (modem.kicad_sch)
- added sheet power_supply (power_supply.kicad_sch)
- added sheet sensor (sensor.kicad_sch)
- added sheet storage (storage.kicad_sch)
- added sheet watchdog (watchdog.kicad_sch)
