File: indicator.kicad_sch (KiCad schematic)
At the start: 15 parts, among them Q5 MMBT2222A, Q6 MMBT2222A, Q7 MMBT2222A

Commit message: adding datasheet
Other:
- note added: "Indicator"
Changed lines of the file:
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@@
 	(generator_version "9.0")
 	(paper "A4")
+	(text "Indicator"
+		(exclude_from_sim no)
+		(at 62.738 60.706 0)
+		(effects
+			(font
+				(size 1.27 1.27)
+			)
+			(justify left)
+		)
+	)
 	(junction
 		(at 149.86 97.79)
@@
 		)
 	)
+	(rule_area
+		(polyline
+			(pts
+				(xy 59.69 57.15) (xy 240.03 57.15) (xy 240.03 116.84) (xy 59.69 116.84)
+			)
+			(stroke
+				(width 0)
+				(type dash)
+			)
+			(fill
+				(type none)
+			)
+		)
+	)
