File: mcu.kicad_sch (KiCad schematic)
At the start: 23 parts, among them J1 USB_B_Micro, J2 PRG, U1 STM32L412CBTxP, Y1 32,768KHz, Y2 16MHz

Commit message: Layout was finish
Changed lines of the file:
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@@
 	)
 	(junction
+		(at 161.29 34.29)
+		(diameter 0)
+		(color 0 0 0 0)
+	)
+	(junction
 		(at 48.26 111.76)
 		(diameter 0)
@@
 	(wire
 		(pts
+			(xy 161.29 33.02) (xy 161.29 34.29)
+		)
+		(stroke
+			(width 0)
+			(type default)
+		)
+	)
+	(wire
+		(pts
 			(xy 220.98 101.6) (xy 223.52 101.6)
 		)
@@
 		(on_board yes)
 		(dnp no)
-		(property "Reference" "#FLG03"
+		(property "Reference" "#FLG02"
 			(at 111.76 31.115 0)
 			(effects
@@
 			(project "SoilMoistureIoT"
 				(path "/6eae54c6-c206-4dc6-8158-b1e680dd71f0/ad775ff2-1cdf-4c1b-bda6-7abaa696ba2c"
-					(reference "#FLG03")
+					(reference "#FLG02")
 					(unit 1)
 				)
@@
 		(on_board yes)
 		(dnp no)
-		(property "Reference" "#FLG02"
+		(property "Reference" "#FLG01"
 			(at 82.55 31.115 0)
 			(effects
@@
 			(project "SoilMoistureIoT"
 				(path "/6eae54c6-c206-4dc6-8158-b1e680dd71f0/ad775ff2-1cdf-4c1b-bda6-7abaa696ba2c"
-					(reference "#FLG02")
+					(reference "#FLG01")
 					(unit 1)
 				)
@@
 	)
 	(symbol
+		(lib_id "power:PWR_FLAG")
+		(at 161.29 33.02 0)
+		(unit 1)
+		(exclude_from_sim no)
+		(in_bom yes)
+		(on_board yes)
+		(dnp no)
+		(property "Reference" "#FLG010"
+			(at 161.29 31.115 0)
+			(effects
+				(font
+					(size 1.27 1.27)
+				)
+				(hide yes)
+			)
+		)
+		(property "Value" "PWR_FLAG"
+			(at 161.29 29.21 0)
+			(effects
+				(font
+					(size 1.27 1.27)
+				)
+			)
+		)
+		(property "Footprint" ""
+			(at 161.29 33.02 0)
+			(effects
+				(font
+					(size 1.27 1.27)
+				)
+				(hide yes)
+			)
+		)
+		(property "Datasheet" "~"
+			(at 161.29 33.02 0)
+			(effects
+				(font
+					(size 1.27 1.27)
+				)
+				(hide yes)
+			)
+		)
+		(property "Description" "Special symbol for telling ERC where power comes from"
+			(at 161.29 33.02 0)
+			(effects
+				(font
+					(size 1.27 1.27)
+				)
+				(hide yes)
+			)
+		)
+		(pin "1"
+		)
+		(instances
+			(project "SoilMoistureIoT"
+				(path "/6eae54c6-c206-4dc6-8158-b1e680dd71f0/ad775ff2-1cdf-4c1b-bda6-7abaa696ba2c"
+					(reference "#FLG010")
+					(unit 1)
+				)
+			)
+		)
+	)
+	(symbol
 		(lib_id "Device:C")
 		(at 146.05 40.64 0)
@@
 		(on_board yes)
 		(dnp no)
-		(property "Reference" "#FLG013"
+		(property "Reference" "#FLG03"
 			(at 195.58 59.055 0)
 			(effects
@@
 			(project "SoilMoistureIoT"
 				(path "/6eae54c6-c206-4dc6-8158-b1e680dd71f0/ad775ff2-1cdf-4c1b-bda6-7abaa696ba2c"
-					(reference "#FLG013")
+					(reference "#FLG03")
 					(unit 1)
 				)

Commit message: adding datasheet
Other:
- note added: "HSE 16MHz (Main clock source)"
- note added: "LSE 32,768KHz (RTC clock source)"
- note added: "MCU decoupling capacitor"
- note added: "Programing line"
- note added: "Universal Serial Bus"
- moved on the sheet: C1, C10, C11, C12, C13, C14, C2, C3, C4, C5, C6, C7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
