File: modem.kicad_sch (KiCad schematic)
At the start: 36 parts, among them J3 Conn_Coaxial, Q1 DTC043ZEBTL, Q2 DTC043ZEBTL, Q3 MMBT2222A, Q4 MMBT2222A, U2 BG95M3LA-64-SGNS

Commit message: adding datasheet
Other:
- note added: "GSM Antena"
- note added: "Modem ~{reset}"
- note added: "R13, C16 and C17 is for impedance tunning"
- note added: "Serial UART"
- note added: "~{Power key}"
- moved on the sheet: C15, C16, C17, C18, C19, J3, Q1, Q2, Q3, Q4, R10, R11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
