File: power_supply.kicad_sch (KiCad schematic)
At the start: 17 parts, among them J6 Battery, U10 TPS61070DDCR, U6 LDO40LPU33RY, U7 BQ25180YBGR, U8 TLV76733DRVR, U9 LDO40LPU33RY

Commit message: Layout was finish
Parts:
- removed C40, C41: C_Polarized, Capacitor_SMD:CP_Elec_6.3x5.7, symbol Device:C_Polarized
- removed U9: LDO40LPU33RY, Package_DFN_QFN:DFN-6-1EP_3x3mm_P0.95mm_EP1.7x2.6mm, symbol Regulator_Linear:LDO40LPU33RY
- added C36, C39: 1u, Capacitor_SMD:C_0402_1005Metric, symbol Device:C
- added C40: 10u, Capacitor_SMD:C_0402_1005Metric, symbol Device:C
- added Q8: DTC043ZEBTL, DTC043ZEBTL:SOTFL50P160X85-3N, symbol DTC043ZEBTL:DTC043ZEBTL
- added R45, R46: 10k, Resistor_SMD:R_0402_1005Metric, symbol Device:R
- renumbered C36 to C37, C37 to C38, C38 to C41, C39 to C42, C42 to C43, C43 to C44, R45 to R47, R46 to R48, U10 to U9
Connections:
- net BATTERY: now also C39.1
- net GND: now also C36.2, C39.2, C40.2, R46.1
- net SYS: now also C40.1
- net VBUS: now also C36.1, R45.2
- net VDD_3V3: now also Q8.3
- net VDD_USB: now also Q8.2
- new net: Q8.1, R45.1, R46.2
Other:
- moved on the sheet: U7

Commit message: adding datasheet
Other:
- note added: "Battery connector"
Changed lines of the file:
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@@
 	(generator_version "9.0")
 	(paper "A4")
+	(text "Battery connector"
+		(exclude_from_sim no)
+		(at 220.472 43.688 0)
+		(effects
+			(font
+				(size 1.27 1.27)
+			)
+			(justify left)
+		)
+	)
 	(junction
 		(at 207.01 143.51)
@@
 		)
 	)
+	(rule_area
+		(polyline
+			(pts
+				(xy 218.44 40.64) (xy 255.27 40.64) (xy 255.27 68.58) (xy 218.44 68.58)
+			)
+			(stroke
+				(width 0)
+				(type dash)
+			)
+			(fill
+				(type none)
+			)
+		)
+	)
