File: sensor.kicad_sch (KiCad schematic)
At the start: 4 parts, among them J5 Conn_01x03

Commit message: adding datasheet
Other:
- note added: "Analog sensor"
Changed lines of the file:
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@@
+		)
+	)
+	(text "Analog sensor"
+		(exclude_from_sim no)
+		(at 92.964 82.804 0)
+		(effects
+			(font
+				(size 1.27 1.27)
+			)
+			(justify left)
 		)
 	)
@@
 		)
 	)
+	(rule_area
+		(polyline
+			(pts
+				(xy 90.17 78.74) (xy 181.61 78.74) (xy 181.61 125.73) (xy 90.17 125.73)
+			)
+			(stroke
+				(width 0)
+				(type dash)
+			)
+			(fill
+				(type none)
+			)
+		)
+	)
