File: storage.kicad_sch (KiCad schematic)
At the start: 1 part, among them U4 FM25V02A-GTR

Commit message: adding datasheet
Other:
- note added: "Additional storage"
Changed lines of the file:
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@@
 	(generator_version "9.0")
 	(paper "A4")
+	(text "Additional storage"
+		(exclude_from_sim no)
+		(at 115.316 75.438 0)
+		(effects
+			(font
+				(size 1.27 1.27)
+			)
+			(justify left)
+		)
+	)
 	(wire
 		(pts
@@
 		)
 	)
+	(rule_area
+		(polyline
+			(pts
+				(xy 113.03 72.39) (xy 186.69 72.39) (xy 186.69 123.19) (xy 113.03 123.19)
+			)
+			(stroke
+				(width 0)
+				(type dash)
+			)
+			(fill
+				(type none)
+			)
+		)
+	)
