File: usim.kicad_sch (KiCad schematic)
At the start: 10 parts, among them J4 SIM8066-6-1-14-01-A_REVA, U3 IP4220CZ6F

Commit message: adding datasheet
Other:
- note added: "GSM SIM Card connector"
- note added: "SIM Connector TVS"
Changed lines of the file:
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@@
 	(generator_version "9.0")
 	(paper "A4")
+	(text "SIM Connector TVS\n"
+		(exclude_from_sim no)
+		(at 167.894 43.18 0)
+		(effects
+			(font
+				(size 1.27 1.27)
+			)
+			(justify left)
+		)
+	)
+	(text "GSM SIM Card connector\n"
+		(exclude_from_sim no)
+		(at 90.678 78.232 0)
+		(effects
+			(font
+				(size 1.27 1.27)
+			)
+			(justify left)
+		)
+	)
 	(junction
 		(at 125.73 105.41)
@@
 		)
 	)
+	(rule_area
+		(polyline
+			(pts
+				(xy 226.06 40.64) (xy 226.06 72.39) (xy 166.37 72.39) (xy 166.37 40.64)
+			)
+			(stroke
+				(width 0)
+				(type dash)
+			)
+			(fill
+				(type none)
+			)
+		)
+	)
+	(rule_area
+		(polyline
+			(pts
+				(xy 88.9 74.93) (xy 226.06 74.93) (xy 226.06 133.35) (xy 88.9 133.35)
+			)
+			(stroke
+				(width 0)
+				(type dash)
+			)
+			(fill
+				(type none)
+			)
+		)
+	)
