File: v_batt.kicad_sch (KiCad schematic)
At the start: 16 parts

Commit message: adding datasheet
Other:
- note added: "Modem decoupling capacitor"
Changed lines of the file:
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@@
 	(generator_version "9.0")
 	(paper "A4")
+	(text "Modem decoupling capacitor"
+		(exclude_from_sim no)
+		(at 55.88 61.722 0)
+		(effects
+			(font
+				(size 1.27 1.27)
+			)
+			(justify left)
+		)
+	)
 	(junction
 		(at 181.61 105.41)
@@
 		)
 	)
+	(rule_area
+		(polyline
+			(pts
+				(xy 53.34 57.15) (xy 266.7 57.15) (xy 266.7 115.57) (xy 53.34 115.57)
+			)
+			(stroke
+				(width 0)
+				(type dash)
+			)
+			(fill
+				(type none)
+			)
+		)
+	)
