File: watchdog.kicad_sch (KiCad schematic)
At the start: 2 parts, among them U5 TPS3431SDRBR

Commit message: adding datasheet
Other:
- note added: "External watchdog"
Changed lines of the file:
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@@
 	(generator_version "9.0")
 	(paper "A4")
+	(text "External watchdog"
+		(exclude_from_sim no)
+		(at 104.902 78.486 0)
+		(effects
+			(font
+				(size 1.27 1.27)
+			)
+			(justify left)
+		)
+	)
 	(junction
 		(at 168.91 99.06)
@@
 		)
 	)
+	(rule_area
+		(polyline
+			(pts
+				(xy 102.87 74.93) (xy 186.69 74.93) (xy 186.69 120.65) (xy 102.87 120.65)
+			)
+			(stroke
+				(width 0)
+				(type dash)
+			)
+			(fill
+				(type none)
+			)
+		)
+	)
